File: hw/kegboard-coaster/kegboard-coaster-v2/kegboard-coaster.sch (EAGLE design)
At the start: 8 parts

Commit message: Replace Temp Sensor with SMD package
Parts:
- removed U$1: TEMPERATURE-SENSOR, geoffculp:TEMPERATURE-SENSOR
- added U$2: TEMPERATURE-SENSORUMAX8, geoffculp:TEMPERATURE-SENSORUMAX8
Connections:
- net 5V: now also U$2.VCC; no longer U$1.VCC
- net GND: now also U$2.GND; no longer U$1.GND
- net ONEWIRE_A: now also U$2.DQ; no longer U$1.DQ
Changed lines of the file:
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@@
 <part name="J_OW" library="SparkFun-20100412" deviceset="M06" device="SIP"/>
 <part name="J_OW1" library="SparkFun-20100412" deviceset="M06" device="SIP"/>
-<part name="U$1" library="geoffculp" deviceset="TEMPERATURE-SENSOR" device=""/>
 <part name="R1" library="resistor" deviceset="R-US_" device="R0805" value="1K"/>
 <part name="LED1" library="SparkFun-LED" deviceset="LED" device="-FKIT-1206"/>
 <part name="C1" library="SparkFun-Passives" deviceset="CAP" device="0805" value="0.1 uF"/>
+<part name="U$2" library="geoffculp" deviceset="TEMPERATURE-SENSOR" device="UMAX8"/>
 </parts>
 <sheets>
@@
 <instance part="J_OW" gate="G$1" x="172.72" y="121.92" rot="R180"/>
 <instance part="J_OW1" gate="G$1" x="172.72" y="96.52" rot="R180"/>
-<instance part="U$1" gate="G$1" x="106.68" y="106.68"/>
 <instance part="R1" gate="G$1" x="45.72" y="104.14"/>
 <instance part="LED1" gate="G$1" x="58.42" y="104.14" rot="R90"/>
 <instance part="C1" gate="G$1" x="60.96" y="83.82"/>
+<instance part="U$2" gate="G$1" x="106.68" y="106.68"/>
 </instances>
 <busses>
@@
 <wire x1="137.16" y1="106.68" x2="116.84" y2="106.68" width="0.1524" layer="91"/>
 <label x="121.92" y="106.68" size="1.778" layer="95"/>
-<pinref part="U$1" gate="G$1" pin="DQ"/>
+<pinref part="U$2" gate="G$1" pin="DQ"/>
 </segment>
 <segment>
@@
 <wire x1="99.06" y1="109.22" x2="86.36" y2="109.22" width="0.1524" layer="91"/>
 <label x="86.36" y="109.22" size="1.778" layer="95"/>
-<pinref part="U$1" gate="G$1" pin="VCC"/>
+<pinref part="U$2" gate="G$1" pin="VCC"/>
 </segment>
 <segment>
@@
 <wire x1="99.06" y1="104.14" x2="86.36" y2="104.14" width="0.1524" layer="91"/>
 <label x="86.36" y="104.14" size="1.778" layer="95"/>
-<pinref part="U$1" gate="G$1" pin="GND"/>
+<pinref part="U$2" gate="G$1" pin="GND"/>
 </segment>
 <segment>

Commit message: Fix temp. sensor REFDES
Parts:
- renumbered U$2 to U$1
Changed lines of the file:
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@@
 <part name="LED1" library="SparkFun-LED" deviceset="LED" device="-FKIT-1206"/>
 <part name="C1" library="SparkFun-Passives" deviceset="CAP" device="0805" value="0.1 uF"/>
-<part name="U$2" library="geoffculp" deviceset="TEMPERATURE-SENSOR" device="UMAX8"/>
+<part name="U$1" library="geoffculp" deviceset="TEMPERATURE-SENSOR" device="UMAX8"/>
 </parts>
 <sheets>
@@
 <instance part="LED1" gate="G$1" x="58.42" y="104.14" rot="R90"/>
 <instance part="C1" gate="G$1" x="60.96" y="83.82"/>
-<instance part="U$2" gate="G$1" x="106.68" y="106.68"/>
+<instance part="U$1" gate="G$1" x="106.68" y="106.68"/>
 </instances>
 <busses>
@@
 <wire x1="137.16" y1="106.68" x2="116.84" y2="106.68" width="0.1524" layer="91"/>
 <label x="121.92" y="106.68" size="1.778" layer="95"/>
-<pinref part="U$2" gate="G$1" pin="DQ"/>
+<pinref part="U$1" gate="G$1" pin="DQ"/>
 </segment>
 <segment>
@@
 <wire x1="99.06" y1="109.22" x2="86.36" y2="109.22" width="0.1524" layer="91"/>
 <label x="86.36" y="109.22" size="1.778" layer="95"/>
-<pinref part="U$2" gate="G$1" pin="VCC"/>
+<pinref part="U$1" gate="G$1" pin="VCC"/>
 </segment>
 <segment>
@@
 <wire x1="99.06" y1="104.14" x2="86.36" y2="104.14" width="0.1524" layer="91"/>
 <label x="86.36" y="104.14" size="1.778" layer="95"/>
-<pinref part="U$2" gate="G$1" pin="GND"/>
+<pinref part="U$1" gate="G$1" pin="GND"/>
 </segment>
 <segment>
